Commit message: add single_motor config

File: urdf/primitive.urdf.xacro (robot description, xacro)
@@ -129,5 +129,5 @@
             <child link="${child}" />
             <axis xyz="${axis}" />
-            <limit effort="0.0" velocity="0.0"/>
+            <limit effort="${effort}" velocity="${velocity}"/>
             <dynamics damping="${damping}" friction="${friction}" />
         </joint>
